File: pt2399_delay.sch (EAGLE design)
At the start: 25 parts, among them U1 PT2399

Commit message: 0510 amp circuit schematic add
Parts:
- added C1, C17: 10u, Capasitor:C-EUC0805K
- added C15, C16: 100u6.3, Capasitor:CPOL-EUTAP5-45
- added IC1: 4558N, OPAMP:4558N
- added MIX1: 10KB, alps-potentiometers:RK09K113
- added R10, R11, R12, R13: 15K, Resistor:RESISTOR2012/0805
Connections:
- new net N$17: C17.1, MIX1.A, R12.1, R13.2
- new net N$23: IC1A.+IN, IC1B.+IN, MIX1.E
- new net N$24: C16.+, IC1A.-IN, IC1A.OUT
- new net N$25: C16.-, R10.2
- new net N$26: C15.+, IC1B.-IN, IC1B.OUT
- new net N$27: C15.-, R11.2
- net GND: now also C1.1, IC1P.V-, MIX1.S, R12.2
- net VCC: now also C1.2, IC1P.V+, R13.1
Other:
- note added: "Delay"
- moved on the sheet: C10, C11, C12, C13, C14, C2, C3, C4, C5, C6, C7, C8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
